File: H5 FC.kicad_pcb (KiCad board)
At the start: 4 copper layers, 38 x 38 mm, 125 parts, among them J1 Conn_01x04_Pin, J13 Conn_01x06, J14 Conn_01x06, J16 Conn_01x06, J17 Conn_01x06, J2 USB_C_Receptacle_USB2.0_16P, J3 Conn_01x08, J4 Micro_SD_Card, J5 Conn_01x08, J6 Conn_01x03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

Commit message: Add V1.1
Add V1.1

Add V1.1
Parts:
- R14: value 100K -> 105K
- R15: value 12.7K -> 13.3K
- moved J14 0.65 mm to (142.5, 54.7)
Connections:
- net GPIO1~_ADC renamed GPIO4~_ADC
- net GPIO2~_ADC renamed GPIO5~_ADC
- net GPIO3~ renamed GPIO6~
- net GPIO4 renamed GPIO2
- net GPIO5 renamed GPIO3
- net GPIO6 renamed GPIO1
Routing:
- net GPIO4~_ADC: track 48.8 -> 49.9 mm
- net +5V: track 149.2 -> 148.6 mm
Other:
- board text added: "CTS"
- board text added: "RTS"

Commit message: v1.1.1 layout version
v1.1.1 layout version
Parts:
- moved C22 1.51 mm to (143.3, 81.3), turned to 0 degrees
- moved C10 0.85 mm to (143.3, 79.7), turned to 180 degrees
- moved C44 0.41 mm to (141.7, 65.3)
- moved C11 0.14 mm to (150.3, 79.7)
Routing:
- net +3.3V: track 173.6 -> 167.6 mm
- net UART7_RX: track 60.4 -> 64.4 mm
- net UART6_TX: track 31.3 -> 29.5 mm
- net MOT2_PWM: track 10.9 -> 9.75 mm
- net MOT1_PWM: track 12.9 -> 11.7 mm
- net Net-(U1-PC0): track 10.9 -> 10.1 mm
- net I2C1_SDA: track 58.1 -> 57.4 mm
- net Analog_IN1: track 63.8 -> 64.4 mm
- net UART5_TX: track 11.9 -> 11.4 mm
- net GND: track 81.0 -> 80.8 mm, vias 106 -> 109
Other:
- board text added: "V1.1.1"

Commit message: v1.2
v1.2
Parts:
- added R5: 10K, Resistor_SMD:R_0603_1608Metric, B.Cu at (149.5, 64.2)
- added R6: 10K, Resistor_SMD:R_0603_1608Metric, B.Cu at (149.5, 72.8)
- added R7: 10K, Resistor_SMD:R_0603_1608Metric, B.Cu at (147.7, 72.8)
- added R8: 10K, Resistor_SMD:R_0603_1608Metric, B.Cu at (147.6, 64.2)
- added R9: 10K, Resistor_SMD:R_0603_1608Metric, B.Cu at (145.4, 64.2)
- moved C26 0.22 mm to (145.4, 68.1)
Routing:
- net +3.3V: track 167.6 -> 177.7 mm
- net SDMMC_D0: track 11.2 -> 15.5 mm
- net SDMMC_D3: track 6.33 -> 9.20 mm
- net SDMMC_CMD: track 13.8 -> 16.4 mm
- net SDMMC_D1: track 13.2 -> 15.3 mm
- net GND: track 80.8 -> 82.7 mm, vias 109 -> 100
- net UART6_RX: track 38.2 -> 39.6 mm
- net SDMMC_D2: track 6.97 -> 8.12 mm
Other:
- board text added: "V1.2.1"
- board text removed: "V1.1.1"

Commit message: Improve board
Routing:
- net SDMMC_CK: track 4.37 -> 10.8 mm
- net SDMMC_D3: track 9.20 -> 15.6 mm
- net SDMMC_D2: track 8.12 -> 12.8 mm
- net GND: track 82.7 -> 85.6 mm, vias 100 -> 99
