File: connectors.kicad_sch (KiCad schematic)
At the start: 25 parts, among them J1 Conn_01x04_Pin, J13 Conn_01x06, J14 Conn_01x06, J16 Conn_01x06, J17 Conn_01x06, J2 USB_C_Receptacle_USB2.0_16P, J3 Conn_01x08, J4 Micro_SD_Card, J5 Conn_01x08, J6 Conn_01x03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

Commit message: Add V1.1
Add V1.1

Add V1.1
Connections:
- net GPIO1~_ADC renamed GPIO4~_ADC
- net GPIO2~_ADC renamed GPIO5~_ADC
- net GPIO3~ renamed GPIO6~
- net GPIO4 renamed GPIO2
- net GPIO5 renamed GPIO3
- net GPIO6 renamed GPIO1
Changed lines of the file:
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@@
 	(title_block
 		(title "STM32H5 FC")
-		(date "08/06/2026")
-		(rev "v1")
+		(date "2026-05-11")
+		(rev "v1.1")
 		(comment 1 "Evans Cesil Thomas")
 	)
@@
 		)
 	)
-	(global_label "GPIO4"
+	(global_label "GPIO2"
 		(shape input)
 		(at 138.43 96.52 0)
@@
 		)
 	)
-	(global_label "GPIO3~"
+	(global_label "GPIO6~"
 		(shape input)
 		(at 176.53 120.65 0)
@@
 		)
 	)
-	(global_label "GPIO6"
+	(global_label "GPIO1"
 		(shape input)
 		(at 176.53 90.17 0)
@@
 		)
 	)
-	(global_label "GPIO2~_ADC"
+	(global_label "GPIO5~_ADC"
 		(shape input)
 		(at 176.53 118.11 0)
@@
 		)
 	)
-	(global_label "GPIO5"
+	(global_label "GPIO3"
 		(shape input)
 		(at 138.43 88.9 0)
@@
 		)
 	)
-	(global_label "GPIO1~_ADC"
+	(global_label "GPIO4~_ADC"
 		(shape input)
 		(at 138.43 93.98 0)

Commit message: v1.2
v1.2
Parts:
- added R5, R6, R7, R8, R9: 10K, Resistor_SMD:R_0603_1608Metric, symbol Device:R_Small
Connections:
- net +3.3V: now also R5.1, R6.1, R7.1, R8.1, R9.1
- net SDMMC_CMD: now also R9.2
- net SDMMC_D0: now also R8.2
- net SDMMC_D1: now also R5.2
- net SDMMC_D2: now also R6.2
- net SDMMC_D3: now also R7.2
Other:
- note removed: "SBUS can be powered with USB"

Commit message: Improve board
Parts:
- R5, R6, R7, R8, R9: value 10K -> 47K
Connections:
- net GPIO2 renamed GPIO2~
Changed lines of the file:
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@@
 		)
 	)
-	(global_label "GPIO2"
+	(global_label "GPIO2~"
 		(shape input)
 		(at 138.43 96.52 0)
@@
 		)
 		(property "Intersheetrefs" "${INTERSHEET_REFS}"
-			(at 147.1 96.52 0)
+			(at 148.0071 96.52 0)
 			(hide yes)
 			(show_name no)
@@
 			)
 		)
-		(property "Value" "10K"
+		(property "Value" "47K"
 			(at 261.62 36.8299 0)
 			(show_name no)
@@
 			)
 		)
-		(property "Value" "10K"
+		(property "Value" "47K"
 			(at 245.11 36.8299 0)
 			(show_name no)
@@
 			)
 		)
-		(property "Value" "10K"
+		(property "Value" "47K"
 			(at 279.4 36.8299 0)
 			(show_name no)
@@
 		(in_pos_files yes)
 		(dnp no)
-		(fields_autoplaced yes)
 		(property "Reference" "R8"
-			(at 254 34.2899 0)
+			(at 254 34.29 0)
 			(show_name no)
 			(do_not_autoplace no)
@@
 			)
 		)
-		(property "Value" "10K"
+		(property "Value" "47K"
 			(at 254 36.8299 0)
 			(show_name no)
-			(do_not_autoplace no)
+			(do_not_autoplace yes)
 			(effects
 				(font
@@
 			)
 		)
-		(property "Value" "10K"
+		(property "Value" "47K"
 			(at 270.51 36.8299 0)
 			(show_name no)
@@
 		)
 	)
-	(embedded_fonts no)
 )
